File: kicad/led_2048/button_board.kicad_pcb (KiCad board)
At the start: 2 copper layers, 80 x 60 mm, 63 parts, among them J10 Power conn, J11 Button conn, J6 Power conn, J7 Mux Conn, J8 Shift Reg Conn, J9 Misc conn 1, SW10 Button, SW11 Button, SW12 Button, SW3 Button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

Commit message: finalized boards and cad files
Parts:
- added REF**: C_0805_2012Metric_Pad1.18x1.45mm_HandSolder, Capacitor_SMD:C_0805_2012Metric_Pad1.18x1.45mm_HandSolder, F.Cu at (114.8, 128.8)
- moved R23 1.01 mm to (114.1, 132.4)
- moved R22 0.16 mm to (109.8, 129.5)
Routing:
- net VDD: track 0.00 -> 1.97 mm
- net GND: track 3.68 -> 5.11 mm, vias 2 -> 3
- net Score data: track 4.57 -> 3.74 mm
- net /Press buttons/Button 1: track 27.8 -> 27.0 mm
