File: kicad/led_2048/display.kicad_sch (KiCad schematic)
At the start: 29 parts, among them U3 TLC59116ITPWRQ1

Commit message: finished layout
Parts:
- C10: value 1uF -> 0.1uF; footprint Capacitor_SMD:C_0805_2012Metric_Pad1.18x1.45mm_HandSolder -> Capacitor_SMD:C_0402_1005Metric_Pad0.74x0.62mm_HandSolder
- renumbered R15 to R14
Changed lines of the file:
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@@
 		(dnp no)
 		(fields_autoplaced yes)
-		(property "Reference" "#PWR030"
+		(property "Reference" "#PWR032"
 			(at 196.85 147.32 0)
 			(effects
@@
 			(project ""
 				(path "/c576df4b-92c0-44b0-b003-b697a5a04765/c77ae034-cca4-473c-b646-c49363a57ea5"
-					(reference "#PWR030")
+					(reference "#PWR032")
 					(unit 1)
 				)
@@
 		(dnp no)
 		(fields_autoplaced yes)
-		(property "Reference" "R15"
+		(property "Reference" "R14"
 			(at 212.09 59.69 90)
 			(effects
@@
 			(project ""
 				(path "/c576df4b-92c0-44b0-b003-b697a5a04765/c77ae034-cca4-473c-b646-c49363a57ea5"
-					(reference "R15")
+					(reference "R14")
 					(unit 1)
 				)
@@
 		(dnp no)
 		(fields_autoplaced yes)
-		(property "Reference" "#PWR027"
+		(property "Reference" "#PWR029"
 			(at 203.2 77.47 0)
 			(effects
@@
 			(project "led_2048"
 				(path "/c576df4b-92c0-44b0-b003-b697a5a04765/c77ae034-cca4-473c-b646-c49363a57ea5"
-					(reference "#PWR027")
+					(reference "#PWR029")
 					(unit 1)
 				)
@@
 		(dnp no)
 		(fields_autoplaced yes)
-		(property "Reference" "#PWR026"
+		(property "Reference" "#PWR028"
 			(at 274.32 63.5 0)
 			(effects
@@
 			(project "led_2048"
 				(path "/c576df4b-92c0-44b0-b003-b697a5a04765/c77ae034-cca4-473c-b646-c49363a57ea5"
-					(reference "#PWR026")
+					(reference "#PWR028")
 					(unit 1)
 				)
@@
 		(dnp no)
 		(fields_autoplaced yes)
-		(property "Reference" "#PWR025"
+		(property "Reference" "#PWR027"
 			(at 261.62 45.72 0)
 			(effects
@@
 			(project "led_2048"
 				(path "/c576df4b-92c0-44b0-b003-b697a5a04765/c77ae034-cca4-473c-b646-c49363a57ea5"
-					(reference "#PWR025")
+					(reference "#PWR027")
 					(unit 1)
 				)
@@
 			)
 		)
-		(property "Value" "1uF"
+		(property "Value" "0.1uF"
 			(at 265.43 59.6899 0)
 			(effects
@@
 			)
 		)
-		(property "Footprint" "Capacitor_SMD:C_0805_2012Metric_Pad1.18x1.45mm_HandSolder"
+		(property "Footprint" "Capacitor_SMD:C_0402_1005Metric_Pad0.74x0.62mm_HandSolder"
 			(at 262.5852 62.23 0)
 			(effects
@@
 		(dnp no)
 		(fields_autoplaced yes)
-		(property "Reference" "#PWR029"
+		(property "Reference" "#PWR031"
 			(at 259.08 110.49 0)
 			(effects
@@
 			(project "led_2048"
 				(path "/c576df4b-92c0-44b0-b003-b697a5a04765/c77ae034-cca4-473c-b646-c49363a57ea5"
-					(reference "#PWR029")
+					(reference "#PWR031")
 					(unit 1)
 				)
@@
 		(dnp no)
 		(fields_autoplaced yes)
-		(property "Reference" "#PWR028"
+		(property "Reference" "#PWR030"
 			(at 218.44 110.49 0)
 			(effects
@@
 			(project ""
 				(path "/c576df4b-92c0-44b0-b003-b697a5a04765/c77ae034-cca4-473c-b646-c49363a57ea5"
-					(reference "#PWR028")
-					(unit 1)
-				)
+					(reference "#PWR030")
+					(unit 1)
+				)

Commit message: finalized boards and cad files
Parts:
- C10: LCSC (none) -> C431646
- D10, D11, D12, D13, D14, D15, D16, D17, D18, D19, D20, D21, D22, D23, D24, D25, D26, D27, D28, D4, D5, D6, D7, D8, D9: footprint LED_THT:LED_D5.0mm-4_RGB -> 2048_footprints:LED_D5.0mm-4x0.8mm_RGB
Changed lines of the file:
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@@
 			)
 		)
-		(property "Footprint" "LED_THT:LED_D5.0mm-4_RGB"
+		(property "Footprint" "2048_footprints:LED_D5.0mm-4x0.8mm_RGB"
 			(at 39.37 63.5 0)
 			(effects
@@
 			)
 		)
-		(property "Footprint" "LED_THT:LED_D5.0mm-4_RGB"
+		(property "Footprint" "2048_footprints:LED_D5.0mm-4x0.8mm_RGB"
 			(at 39.37 114.3 0)
 			(effects
@@
 			)
 		)
-		(property "Footprint" "LED_THT:LED_D5.0mm-4_RGB"
+		(property "Footprint" "2048_footprints:LED_D5.0mm-4x0.8mm_RGB"
 			(at 171.45 38.1 0)
 			(effects
@@
 			)
 		)
-		(property "Footprint" "LED_THT:LED_D5.0mm-4_RGB"
+		(property "Footprint" "2048_footprints:LED_D5.0mm-4x0.8mm_RGB"
 			(at 105.41 139.7 0)
 			(effects
@@
 			)
 		)
-		(property "Footprint" "LED_THT:LED_D5.0mm-4_RGB"
+		(property "Footprint" "2048_footprints:LED_D5.0mm-4x0.8mm_RGB"
 			(at 39.37 38.1 0)
 			(effects
@@
 			)
 		)
-		(property "Footprint" "LED_THT:LED_D5.0mm-4_RGB"
+		(property "Footprint" "2048_footprints:LED_D5.0mm-4x0.8mm_RGB"
 			(at 171.45 114.3 0)
 			(effects
@@
 			)
 		)
-		(property "Footprint" "LED_THT:LED_D5.0mm-4_RGB"
+		(property "Footprint" "2048_footprints:LED_D5.0mm-4x0.8mm_RGB"
 			(at 171.45 63.5 0)
 			(effects
@@
 			)
 		)
-		(property "Footprint" "LED_THT:LED_D5.0mm-4_RGB"
+		(property "Footprint" "2048_footprints:LED_D5.0mm-4x0.8mm_RGB"
 			(at 138.43 38.1 0)
 			(effects
@@
 			)
 		)
-		(property "Footprint" "LED_THT:LED_D5.0mm-4_RGB"
+		(property "Footprint" "2048_footprints:LED_D5.0mm-4x0.8mm_RGB"
 			(at 72.39 88.9 0)
 			(effects
@@
 			)
 		)
-		(property "Footprint" "LED_THT:LED_D5.0mm-4_RGB"
+		(property "Footprint" "2048_footprints:LED_D5.0mm-4x0.8mm_RGB"
 			(at 171.45 88.9 0)
 			(effects
@@
 			)
 		)
-		(property "Footprint" "LED_THT:LED_D5.0mm-4_RGB"
+		(property "Footprint" "2048_footprints:LED_D5.0mm-4x0.8mm_RGB"
 			(at 138.43 139.7 0)
 			(effects
@@
 			)
 		)
-		(property "Footprint" "LED_THT:LED_D5.0mm-4_RGB"
+		(property "Footprint" "2048_footprints:LED_D5.0mm-4x0.8mm_RGB"
 			(at 72.39 38.1 0)
 			(effects
@@
 			)
 		)
-		(property "Footprint" "LED_THT:LED_D5.0mm-4_RGB"
+		(property "Footprint" "2048_footprints:LED_D5.0mm-4x0.8mm_RGB"
 			(at 138.43 114.3 0)
 			(effects
@@
 			)
 		)
-		(property "Footprint" "LED_THT:LED_D5.0mm-4_RGB"
+		(property "Footprint" "2048_footprints:LED_D5.0mm-4x0.8mm_RGB"
 			(at 105.41 88.9 0)
 			(effects
@@
 			)
 		)
-		(property "Footprint" "LED_THT:LED_D5.0mm-4_RGB"
+		(property "Footprint" "2048_footprints:LED_D5.0mm-4x0.8mm_RGB"
 			(at 138.43 63.5 0)
 			(effects
@@
 			)
 		)
+		(property "LCSC" "C431646"
+			(at 261.62 58.42 0)
+			(effects
+				(font
+					(size 1.27 1.27)
+				)
+				(hide yes)
+			)
+		)
 		(pin "2"
 		)
@@
 			)
 		)
-		(property "Datasheet" "https://item.szlcsc.com/191765.html"
+		(property "Datasheet" "https://www.ti.com/lit/ds/symlink/tlc59116-q1.pdf?ts=1723061996587&ref_url=https%253A%252F%252Fwww.ti.com%252Fproduct%252FTLC59116-Q1%252Fpart-details%252FTLC59116ITPWRQ1%253Fbm-verify%253DAAQAAAAJ_____69QKPd5Itn_pAggT7eJNdg_7UVTr4kMtfmGunJ_E1qWZM59lGjmWXDS10Y-4DMf-VTlYnjgEZUb8MZtYGMUZNrqy3r_7nOvQrETaIoJL_yMrJwMOIV91USEwTpMw2DLk8kZwCSeCM9PlJzb4U6bVyEPvuopbh6r39AAdK8MF3X_SP3DT-S77HIRUALvuu622Q6960lrSrmNWtQGHB-5b5k0fK4yu98M_8Q_aSpB3pdis0vlHGq1hTcvn79nWoTGTIFNFFqpYqdwnogziH66dkZMvm5EJbcRYNhUMR8zVKpi2Btg0vIi4att2orZ7UAyarfNXvraZvwkvurfY90rla1_nOtSFkEk"
 			(at 236.474 83.693 0)
 			(effects
@@
 			)
 		)
-		(property "Footprint" "LED_THT:LED_D5.0mm-4_RGB"
+		(property "Footprint" "2048_footprints:LED_D5.0mm-4x0.8mm_RGB"
 			(at 105.41 38.1 0)
 			(effects
@@
 			)
 		)
-		(property "Footprint" "LED_THT:LED_D5.0mm-4_RGB"
+		(property "Footprint" "2048_footprints:LED_D5.0mm-4x0.8mm_RGB"
 			(at 39.37 139.7 0)
 			(effects
@@
 			)
 		)
-		(property "Footprint" "LED_THT:LED_D5.0mm-4_RGB"
+		(property "Footprint" "2048_footprints:LED_D5.0mm-4x0.8mm_RGB"
 			(at 105.41 114.3 0)
 			(effects
@@
 			)
 		)
-		(property "Footprint" "LED_THT:LED_D5.0mm-4_RGB"
+		(property "Footprint" "2048_footprints:LED_D5.0mm-4x0.8mm_RGB"
 			(at 105.41 63.5 0)
 			(effects
@@
 			)
 		)
-		(property "Footprint" "LED_THT:LED_D5.0mm-4_RGB"
+		(property "Footprint" "2048_footprints:LED_D5.0mm-4x0.8mm_RGB"
 			(at 72.39 114.3 0)
 			(effects
@@
 			)
 		)
-		(property "Footprint" "LED_THT:LED_D5.0mm-4_RGB"
+		(property "Footprint" "2048_footprints:LED_D5.0mm-4x0.8mm_RGB"
 			(at 72.39 139.7 0)
 			(effects
@@
 			)
 		)
-		(property "Footprint" "LED_THT:LED_D5.0mm-4_RGB"
+		(property "Footprint" "2048_footprints:LED_D5.0mm-4x0.8mm_RGB"
 			(at 72.39 63.5 0)
 			(effects
@@
 			)
 		)
-		(property "Footprint" "LED_THT:LED_D5.0mm-4_RGB"
+		(property "Footprint" "2048_footprints:LED_D5.0mm-4x0.8mm_RGB"
 			(at 39.37 88.9 0)
 			(effects
@@
 			)
 		)
-		(property "Footprint" "LED_THT:LED_D5.0mm-4_RGB"
+		(property "Footprint" "2048_footprints:LED_D5.0mm-4x0.8mm_RGB"
 			(at 138.43 88.9 0)
 			(effects
@@
 			)
 		)
-		(property "Footprint" "LED_THT:LED_D5.0mm-4_RGB"
+		(property "Footprint" "2048_footprints:LED_D5.0mm-4x0.8mm_RGB"
 			(at 171.45 139.7 0)
 			(effects

Commit message: minor schematic revisions
Parts:
- renumbered R14 to R16
Changed lines of the file:
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@@
 		(dnp no)
 		(fields_autoplaced yes)
-		(property "Reference" "#PWR032"
+		(property "Reference" "#PWR033"
 			(at 196.85 147.32 0)
 			(effects
@@
 			(project ""
 				(path "/c576df4b-92c0-44b0-b003-b697a5a04765/c77ae034-cca4-473c-b646-c49363a57ea5"
-					(reference "#PWR032")
+					(reference "#PWR033")
 					(unit 1)
 				)
@@
 		(dnp no)
 		(fields_autoplaced yes)
-		(property "Reference" "R14"
+		(property "Reference" "R16"
 			(at 212.09 59.69 90)
 			(effects
@@
 			(project ""
 				(path "/c576df4b-92c0-44b0-b003-b697a5a04765/c77ae034-cca4-473c-b646-c49363a57ea5"
-					(reference "R14")
+					(reference "R16")
 					(unit 1)
 				)
@@
 		(dnp no)
 		(fields_autoplaced yes)
-		(property "Reference" "#PWR029"
+		(property "Reference" "#PWR030"
 			(at 203.2 77.47 0)
 			(effects
@@
 			(project "led_2048"
 				(path "/c576df4b-92c0-44b0-b003-b697a5a04765/c77ae034-cca4-473c-b646-c49363a57ea5"
-					(reference "#PWR029")
+					(reference "#PWR030")
 					(unit 1)
 				)
@@
 		(dnp no)
 		(fields_autoplaced yes)
-		(property "Reference" "#PWR028"
+		(property "Reference" "#PWR029"
 			(at 274.32 63.5 0)
 			(effects
@@
 			(project "led_2048"
 				(path "/c576df4b-92c0-44b0-b003-b697a5a04765/c77ae034-cca4-473c-b646-c49363a57ea5"
-					(reference "#PWR028")
+					(reference "#PWR029")
 					(unit 1)
 				)
@@
 		(dnp no)
 		(fields_autoplaced yes)
-		(property "Reference" "#PWR027"
+		(property "Reference" "#PWR028"
 			(at 261.62 45.72 0)
 			(effects
@@
 			(project "led_2048"
 				(path "/c576df4b-92c0-44b0-b003-b697a5a04765/c77ae034-cca4-473c-b646-c49363a57ea5"
-					(reference "#PWR027")
+					(reference "#PWR028")
 					(unit 1)
 				)
@@
 		(dnp no)
 		(fields_autoplaced yes)
-		(property "Reference" "#PWR031"
+		(property "Reference" "#PWR032"
 			(at 259.08 110.49 0)
 			(effects
@@
 			(project "led_2048"
 				(path "/c576df4b-92c0-44b0-b003-b697a5a04765/c77ae034-cca4-473c-b646-c49363a57ea5"
-					(reference "#PWR031")
+					(reference "#PWR032")
 					(unit 1)
 				)
@@
 		(dnp no)
 		(fields_autoplaced yes)
-		(property "Reference" "#PWR030"
+		(property "Reference" "#PWR031"
 			(at 218.44 110.49 0)
 			(effects
@@
 			(project ""
 				(path "/c576df4b-92c0-44b0-b003-b697a5a04765/c77ae034-cca4-473c-b646-c49363a57ea5"
-					(reference "#PWR030")
-					(unit 1)
-				)
+					(reference "#PWR031")
+					(unit 1)
+				)
