File: kicad/led_2048/led_2048.kicad_pcb (KiCad board)
At the start: 4 copper layers, 47 x 50 mm, 111 parts, among them J1 Program Conn, Q1 PNP, Q2 PNP, Q3 PNP, Q4 PNP, Q5 PNP, SW1 Power switch, SW10 Up, SW2 SW_Push, SW3 Right, SW4 Left, SW5 Down, SW6 B button, SW7 A button, SW8 R button, SW9 L button, U1 TPS73701DRVR, U2 STM32F303CBTx, U3 TLC59116ITPWRQ1, U4 74HC595, U5 CL3641BH

Commit message: finished layout
Parts:
- removed the ? at (354.2, 117.8)
- removed the ? at (394.8, 74.2)
- removed C11, C12, C13, C14, C15, C16, C17, C18: 0.1uF (DNP), Capacitor_SMD:C_0805_2012Metric_Pad1.18x1.45mm_HandSolder
- removed the R1 at (409.7, 126.5)
- removed R16, R17, R18, R19, R20, R21, R22: 220R, Resistor_SMD:R_0805_2012Metric_Pad1.20x1.40mm_HandSolder
- removed R23, R25, R27, R29, R31, R33, R35, R37: 4.7k, Resistor_SMD:R_0805_2012Metric_Pad1.20x1.40mm_HandSolder
- removed R24, R26, R28, R30, R32, R34, R36, R38: 100R (DNP), Resistor_SMD:R_0805_2012Metric_Pad1.20x1.40mm_HandSolder
- removed the REF** at (449.4, 61.9)
- removed SW10: Up, 2048_footprints:SW_TL1105SPF160Q
- removed SW3: Right, 2048_footprints:SW_TL1105SPF160Q
- removed SW4: Left, 2048_footprints:SW_TL1105SPF160Q
- removed SW5: Down, 2048_footprints:SW_TL1105SPF160Q
- removed SW6: B button, 2048_footprints:SW_TL1105SPF160Q
- removed SW7: A button, 2048_footprints:SW_TL1105SPF160Q
- removed SW8: R button, 2048_footprints:SW_TL1105SPF160Q
- removed SW9: L button, 2048_footprints:SW_TL1105SPF160Q
- removed U4: 74HC595, Package_SO:SOP-16_3.9x9.9mm_P1.27mm
- removed U5: CL3641BH, 2048_footprints:CL3641BH
- added ?: , , F.Cu at (218.1, 92.8)
- added ?: , , F.Cu at (218.1, 94.8)
- added H1: MountingHole, MountingHole:MountingHole_3.2mm_M3, F.Cu at (180.1, 93.5)
- added H2: MountingHole, MountingHole:MountingHole_3.2mm_M3, F.Cu at (223.3, 50.3)
- added J12: Shift Reg Conn, Connector_PinSocket_2.00mm:PinSocket_1x03_P2.00mm_Vertical, F.Cu at (224.1, 62.9)
- added J2: Button conn left, 2048_footprints:PinSocket_2x02_P2.00mm_Vertical, B.Cu at (180.8, 87.9)
- added J3: Button conn left, 2048_footprints:PinSocket_2x02_P2.00mm_Vertical, B.Cu at (215.6, 93.8)
- added J4: Misc conn 1, Connector_PinSocket_2.00mm:PinSocket_1x02_P2.00mm_Vertical, F.Cu at (182.3, 49.4)
- added J5: Misc conn 2, Connector_PinSocket_2.00mm:PinSocket_1x02_P2.00mm_Vertical, B.Cu at (184.3, 92.9)
- added JP1: 3.3V, Jumper:SolderJumper-2_P1.3mm_Open_TrianglePad1.0x1.5mm, F.Cu at (213.9, 86.5)
- added REF**: PinSocket_1x04_P2.00mm_Vertical, Connector_PinSocket_2.00mm:PinSocket_1x04_P2.00mm_Vertical, B.Cu at (218.7, 55.3)
- added REF**: PinSocket_1x02_P2.00mm_Vertical, Connector_PinSocket_2.00mm:PinSocket_1x02_P2.00mm_Vertical, B.Cu at (218.1, 94.8)
- added REF**: PinSocket_1x02_P2.00mm_Vertical, Connector_PinSocket_2.00mm:PinSocket_1x02_P2.00mm_Vertical, B.Cu at (218.9, 49.3)
- C1, C4, C9: footprint Capacitor_SMD:C_0805_2012Metric_Pad1.18x1.45mm_HandSolder -> Capacitor_SMD:C_0402_1005Metric_Pad0.74x0.62mm_HandSolder
- C10: value 1uF -> 0.1uF; footprint Capacitor_SMD:C_0805_2012Metric_Pad1.18x1.45mm_HandSolder -> Capacitor_SMD:C_0402_1005Metric_Pad0.74x0.62mm_HandSolder; moved to B.Cu
- C2: footprint Capacitor_SMD:C_0805_2012Metric_Pad1.18x1.45mm_HandSolder -> Capacitor_SMD:C_0603_1608Metric_Pad1.08x0.95mm_HandSolder
- C5, C6, C7, C8: moved to F.Cu
- D1: value Red -> Blue
- D3: value Blue -> Red
- R10: renamed from R11; value TBD -> 1k
- R12: renamed from R13; value 1k -> TBD
- R13: renamed from R14; value 1k -> TBD
- R4: renamed from R5; footprint Resistor_SMD:R_0805_2012Metric_Pad1.20x1.40mm_HandSolder -> Resistor_SMD:R_0603_1608Metric_Pad0.98x0.95mm_HandSolder
- R6: renamed from R7; footprint Resistor_SMD:R_0805_2012Metric_Pad1.20x1.40mm_HandSolder -> Resistor_SMD:R_0603_1608Metric_Pad0.98x0.95mm_HandSolder
- R9: renamed from R10; value TBD -> 1k
- moved C3 243.2 mm to (192.3, 85.6), turned to 180 degrees
- moved C4 228.1 mm to (186.9, 95.2), turned to -90 degrees
- moved C5 226.0 mm to (187.9, 87.3), turned to -90 degrees
- moved C6 216.8 mm to (194.1, 88.2), turned to 180 degrees
- moved C7 211.5 mm to (195.6, 91.7)
- moved C8 211.0 mm to (193.1, 91.7)
- moved R5 203.9 mm to (210.5, 87.3), turned to 0 degrees
- moved C10 203.6 mm to (208.4, 89.7), turned to 90 degrees
- moved C1 198.7 mm to (213.1, 85.9), turned to 90 degrees
- moved R4 194.8 mm to (214.6, 85.5), turned to -90 degrees
- moved R6 191.0 mm to (216.4, 83.7), turned to -90 degrees
- moved D3 188.5 mm to (181.0, 83.1)
- moved D2 186.9 mm to (180.9, 77.6)
- moved C9 186.0 mm to (197.9, 91.1), turned to -90 degrees
- moved D1 185.4 mm to (180.9, 72.1)
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- renumbered R2 to R1, R12 to R11, R15 to R14, R3 to R2, R4 to R3, R6 to R5, R8 to R7, R9 to R8
Connections:
- D1 pad 1: unconnected-(D1-K-Pad1) -> /MCU/Green LED
- D2 pad 1: unconnected-(D2-K-Pad1) -> /MCU/Blue LED
- D3 pad 1: unconnected-(D3-K-Pad1) -> /MCU/Red LED
- J1 pad 2: /MCU/SWCLK -> GND
- J1 pad 3: GND -> /MCU/SWCLK
- R10 pad 1: VDD -> /MCU/MUX4
- R10 pad 2: SDA -> Net-(Q4-B)
- R11 pad 1: /MCU/MUX3 -> /MCU/MUX5
- R11 pad 2: Net-(Q3-B) -> Net-(Q5-B)
- R12 pad 1: /MCU/MUX4 -> VDD
- R12 pad 2: Net-(Q4-B) -> SCL
- R13 pad 1: /MCU/MUX5 -> VDD
- R13 pad 2: Net-(Q5-B) -> SDA
- R9 pad 1: VDD -> /MCU/MUX3
- R9 pad 2: SCL -> Net-(Q3-B)
- SW1 pad 5: (no net) -> GND
- SW2 pad 1: /MCU/~{RESET} -> GND
- SW2 pad 3: (no net) -> /MCU/~{RESET}
- SW2 pad 4: (no net) -> /MCU/~{RESET}
- U2 pad 10: unconnected-(U2-PA0-Pad10) -> /MCU/Button 5
- U2 pad 11: unconnected-(U2-PA1-Pad11) -> /MCU/Button 6
- U2 pad 12: unconnected-(U2-PA2-Pad12) -> /MCU/Button 7
- U2 pad 13: unconnected-(U2-PA3-Pad13) -> /MCU/Button 8
- U2 pad 18: unconnected-(U2-PB0-Pad18) -> /MCU/Score clk
- U2 pad 19: unconnected-(U2-PB1-Pad19) -> /MCU/Score latch
- U2 pad 2: unconnected-(U2-PC13-Pad2) -> /MCU/Red LED
- U2 pad 20: unconnected-(U2-PB2-Pad20) -> /MCU/Score data
- U2 pad 26: unconnected-(U2-PB13-Pad26) -> /MCU/Misc GPIO 4
- U2 pad 27: unconnected-(U2-PB14-Pad27) -> /MCU/Misc GPIO 3
- U2 pad 28: unconnected-(U2-PB15-Pad28) -> /MCU/Misc GPIO 2
- U2 pad 29: unconnected-(U2-PA8-Pad29) -> /MCU/Misc GPIO 1
- U2 pad 3: unconnected-(U2-PC14-Pad3) -> /MCU/Blue LED
- U2 pad 30: unconnected-(U2-PA9-Pad30) -> /MCU/Button 4
- U2 pad 31: unconnected-(U2-PA10-Pad31) -> /MCU/Button 2
- U2 pad 32: unconnected-(U2-PA11-Pad32) -> /MCU/Button 1
- U2 pad 33: unconnected-(U2-PA12-Pad33) -> /MCU/Button 3
- U2 pad 34: unconnected-(U2-PA13-Pad34) -> /MCU/SWDIO
- U2 pad 37: unconnected-(U2-PA14-Pad37) -> /MCU/SWCLK
- U2 pad 38: unconnected-(U2-PA15-Pad38) -> TLC Reset
- U2 pad 39: unconnected-(U2-PB3-Pad39) -> /MCU/MUX1
- U2 pad 4: unconnected-(U2-PC15-Pad4) -> /MCU/Green LED
- U2 pad 40: unconnected-(U2-PB4-Pad40) -> /MCU/MUX2
- U2 pad 41: unconnected-(U2-PB5-Pad41) -> /MCU/MUX3
- U2 pad 42: unconnected-(U2-PB6-Pad42) -> /MCU/MUX4
- U2 pad 43: unconnected-(U2-PB7-Pad43) -> /MCU/MUX5
- U2 pad 44: unconnected-(U2-BOOT0-Pad44) -> GND
- U2 pad 45: unconnected-(U2-PB8-Pad45) -> SCL
- U2 pad 46: unconnected-(U2-PB9-Pad46) -> SDA
Routing:
- net /MCU/Score latch: track 0.00 -> 64.8 mm, vias 0 -> 1
- net /MCU/Score data: track 0.00 -> 63.1 mm, vias 0 -> 1
- net /MCU/Score clk: track 0.00 -> 63.0 mm, vias 0 -> 1
- net /MCU/~{RESET}: track 0.00 -> 56.5 mm, vias 0 -> 1
- net (no net): track 54.1 -> 0.00 mm
- net /MCU/Misc GPIO 2: track 0.00 -> 51.0 mm, vias 0 -> 1
- net /MCU/Misc GPIO 1: track 0.00 -> 50.7 mm, vias 0 -> 1
- net GND: track 4.86 -> 42.3 mm, vias 3 -> 24
- net /LED Matrix/OUT14: track 12.1 -> 48.0 mm
- net /LED Matrix/OUT12: track 6.65 -> 41.2 mm
- net /MCU/Green LED: track 0.00 -> 33.8 mm, vias 0 -> 1
- net /MCU/Blue LED: track 0.00 -> 27.2 mm, vias 0 -> 1
- net /LED Matrix/OUT13: track 10.6 -> 36.7 mm
- net /MCU/MUX3: track 5.14 -> 27.6 mm
- net /MCU/Button 8: track 0.00 -> 21.8 mm
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- added copper zone on B.Cu, net GND
- added copper zone on F.Cu, net GND
- added copper zone on B.Cu, net Net-(JP1-A)
Other:
- board size 47 x 50 mm -> 50 x 50 mm
- board text added: "+"
- board text added: "BAT+ <"
- board text added: "BAT- <"
- board text added: "CLK"
- board text added: "DIO"
- board text added: "GND"
- board text added: "Make RGB led hold size at least 0.8mm Double check the leds that you ordered have a pitch of about 0.5mm!"

Commit message: finalized boards and cad files
Parts:
- removed ? (x2): , 
- added JP2: , 2048_footprints:PinSocket_5x2.54_SMD_90deg_952-3198-1-ND, F.Cu at (180.8, 63.8)
- C2: footprint Capacitor_SMD:C_0603_1608Metric_Pad1.08x0.95mm_HandSolder -> Capacitor_SMD:C_0805_2012Metric_Pad1.18x1.45mm_HandSolder
- C5: footprint Capacitor_SMD:C_0805_2012Metric_Pad1.18x1.45mm_HandSolder -> Capacitor_SMD:C_0402_1005Metric_Pad0.74x0.62mm_HandSolder; moved to B.Cu
- D10, D11, D12, D13, D14, D15, D16, D17, D18, D19, D20, D21, D22, D23, D24, D25, D26, D27, D28, D4, D5, D6, D7, D8, D9: footprint LED_THT:LED_D5.0mm-4_RGB -> 2048_footprints:LED_D5.0mm-4x0.8mm_RGB
- R1, R2, R3: value TBD -> 330R
- R12, R13: value TBD -> 10k
- moved R2 6.65 mm to (188.9, 83.3), turned to 180 degrees
- moved JP1 2.89 mm to (213.4, 89.3), turned to -90 degrees
- moved C5 1.97 mm to (186.6, 85.8), turned to 180 degrees
- moved C3 1.81 mm to (194.1, 85.2)
- moved C1 1.41 mm to (211.8, 85.3), turned to 0 degrees
- moved C2 1.04 mm to (214.1, 89.3)
- moved C6 0.81 mm to (194.1, 87.4)
- moved R4 0.65 mm to (214.1, 85.1)
- moved R6 0.40 mm to (216.4, 83.3)
- moved J1 0.30 mm to (208.7, 92.0)
- moved R5 0.28 mm to (210.2, 87.3)
- moved C10 0.20 mm to (208.4, 89.5)
- moved J3 0.12 mm to (215.6, 93.9)
- moved R13 0.12 mm to (206.2, 85.0)
- moved REF** 0.09 mm to (218.1, 94.7)
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- renumbered REF** to J7
Routing:
- net unconnected-(U2-PA4-Pad14): track 0.00 -> 60.3 mm, vias 0 -> 2
- net unconnected-(U2-PA5-Pad15): track 0.00 -> 59.1 mm, vias 0 -> 2
- net unconnected-(U2-PA6-Pad16): track 0.00 -> 47.8 mm, vias 0 -> 2
- net unconnected-(U2-PA7-Pad17): track 0.00 -> 47.1 mm, vias 0 -> 2
- net unconnected-(U2-PB12-Pad25): track 0.00 -> 34.2 mm, vias 0 -> 2
- net GND: track 42.3 -> 29.7 mm, vias 24 -> 67
- net /MCU/~{RESET}: track 56.5 -> 47.7 mm, vias 1 -> 2
- net Net-(D2-A): track 3.74 -> 11.8 mm
- net VDD: track 45.6 -> 38.8 mm, vias 14 -> 12
- net Multiplex 5: track 46.5 -> 41.2 mm
- net Multiplex 1: track 53.7 -> 49.5 mm
- net Multiplex 3: track 62.8 -> 58.7 mm
- net Net-(SW1-A): track 14.3 -> 11.7 mm, vias 1 -> 0
- net Multiplex 2: track 54.2 -> 52.0 mm
- net Net-(U1-NR/FB): track 5.54 -> 7.10 mm
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- added copper zone on In3.Cu, net GND
- added copper zone on In4.Cu, net GND
- added copper zone on F.Cu, net VDD
Other:
- copper layers 4 -> 6
- board text added: "A4"
- board text added: "A5"
- board text added: "A6"
- board text added: "A7"
- board text added: "B12"
- board text added: "~{NRST}"
- board text removed: "${REFERENCE}"
- board text removed: "Make RGB led hold size at least 0.8mm Double check the leds that you ordered have a pitch of about 0.5mm!"

Commit message: added solderbridge for bootloader
Parts:
- added JP2: Solder Bridge, Jumper:SolderJumper-3_P1.3mm_Open_Pad1.0x1.5mm_NumberLabels, F.Cu at (194.0, 82.8)
- C2: footprint Capacitor_SMD:C_0805_2012Metric_Pad1.18x1.45mm_HandSolder -> Capacitor_SMD:C_0603_1608Metric_Pad1.08x0.95mm_HandSolder
- H1, H2: value MountingHole -> MountingHole M3
Connections:
- U2 pad 44: GND -> /MCU/~{BOOT}
Routing:
- net /MCU/~{BOOT}: track 0.00 -> 4.96 mm, vias 0 -> 1
- net GND: track 29.7 -> 27.1 mm, vias 67 -> 66
- net VDD: track 38.8 -> 37.6 mm

Commit message: minor schematic revisions
Parts:
- removed the JP2 at (194.0, 82.8)
- added R12: 0R (DNP), Resistor_SMD:R_0805_2012Metric_Pad1.20x1.40mm_HandSolder, F.Cu at (194.1, 82.9)
- added R13: 10k, Resistor_SMD:R_0805_2012Metric_Pad1.20x1.40mm_HandSolder, F.Cu at (189.0, 85.4)
- renumbered J4 to J1, J1 to J2, J5 to J3, J12 to J4, J2 to J5, J3 to J6, R12 to R14, R13 to R15, R14 to R16
Routing:
- net /MCU/~{BOOT}: track 4.96 -> 8.39 mm
