File: kicad/led_2048/mcu.kicad_sch (KiCad schematic)
At the start: 39 parts, among them J1 Program Conn, Q1 PNP, Q2 PNP, Q3 PNP, Q4 PNP, Q5 PNP, SW1 Power switch, SW2 SW_Push, U1 TPS73701DRVR, U2 STM32F303CBTx

Commit message: finished layout
Parts:
- removed R1: 0R (DNP), Resistor_SMD:R_0805_2012Metric_Pad1.20x1.40mm_HandSolder, symbol Device:R_US
- added H1, H2: MountingHole, MountingHole:MountingHole_3.2mm_M3, symbol Mechanical:MountingHole
- added J12: Shift Reg Conn, Connector_PinSocket_2.00mm:PinSocket_1x03_P2.00mm_Vertical, symbol Connector:Conn_01x03_Socket
- added J2, J3: Button conn left, 2048_footprints:PinSocket_2x02_P2.00mm_Vertical, symbol Connector:Conn_01x04_Socket
- added J4: Misc conn 1, Connector_PinSocket_2.00mm:PinSocket_1x02_P2.00mm_Vertical, symbol Connector:Conn_01x02_Socket
- added J5: Misc conn 2, Connector_PinSocket_2.00mm:PinSocket_1x02_P2.00mm_Vertical, symbol Connector:Conn_01x02_Socket
- added JP1: 3.3V, Jumper:SolderJumper-2_P1.3mm_Open_TrianglePad1.0x1.5mm, symbol Jumper:SolderJumper_2_Open
- C1, C4, C9: footprint Capacitor_SMD:C_0805_2012Metric_Pad1.18x1.45mm_HandSolder -> Capacitor_SMD:C_0402_1005Metric_Pad0.74x0.62mm_HandSolder
- C2: footprint Capacitor_SMD:C_0805_2012Metric_Pad1.18x1.45mm_HandSolder -> Capacitor_SMD:C_0603_1608Metric_Pad1.08x0.95mm_HandSolder
- R4: renamed from R5; footprint Resistor_SMD:R_0805_2012Metric_Pad1.20x1.40mm_HandSolder -> Resistor_SMD:R_0603_1608Metric_Pad0.98x0.95mm_HandSolder
- R6: renamed from R7; footprint Resistor_SMD:R_0805_2012Metric_Pad1.20x1.40mm_HandSolder -> Resistor_SMD:R_0603_1608Metric_Pad0.98x0.95mm_HandSolder
- SW2: symbol Switch:SW_Push -> Switch:SW_MEC_5E
- renumbered D3 to D1, D1 to D3, R4 to R1, R13 to R10, R14 to R11, R10 to R12, R11 to R13, R3 to R2, R2 to R3, R6 to R5, R8 to R7, R9 to R8, R12 to R9
Connections:
- net Blue LED: now also D2.1 (K), U2.3 (PC14)
- net GND: now also J1.2 (Pin_2), SW1.4 (SH1), SW1.5 (SH2), SW2.1, U2.44 (BOOT0); no longer J1.3 (Pin_3)
- net Green LED: now also D1.1 (K), U2.4 (PC15)
- net MUX1: now also U2.39 (PB3)
- net MUX2: now also U2.40 (PB4)
- net MUX3: now also U2.41 (PB5)
- net MUX4: now also U2.42 (PB6)
- net MUX5: now also U2.43 (PB7)
- net Red LED: now also D3.1 (K), U2.2 (PC13)
- net SCL: now also U2.45 (PB8)
- net SDA: now also U2.46 (PB9)
- net SWCLK: now also J1.3 (Pin_3), U2.37 (PA14); no longer J1.2 (Pin_2)
- net SWDIO: now also U2.34 (PA13)
- net Score clk: now also U2.18 (PB0), J12.3 (Pin_3)
- net Score data: now also U2.20 (PB2), J12.1 (Pin_1)
- net Score latch: now also U2.19 (PB1), J12.2 (Pin_2)
- net TLC Reset: now also U2.38 (PA15)
- net VDD: now also JP1.2 (B)
- net ~{RESET}: now also SW2.3 (K), SW2.4 (A); no longer SW2.1
- net at C1.1, C2.1, R4.2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: now also JP1.1 (A)
- net Button 5: now reaches U2.10 (PA0)
- net Button 5: now also J3.1 (Pin_1)
- net Button 6: now reaches U2.11 (PA1)
- net Button 6: now also J3.2 (Pin_2)
- net Button 7: now reaches U2.12 (PA2)
- net Button 7: now also J3.3 (Pin_3)
- net Button 8: now reaches U2.13 (PA3)
- net Button 8: now also J3.4 (Pin_4)
- net Misc GPIO 4: now reaches U2.26 (PB13)
- net Misc GPIO 4: now also J5.2 (Pin_2)
- net Misc GPIO 3: now reaches U2.27 (PB14)
- net Misc GPIO 3: now also J5.1 (Pin_1)
- net Misc GPIO 2: now reaches U2.28 (PB15)
- net Misc GPIO 2: now also J4.2 (Pin_2)
- net Misc GPIO 1: now reaches U2.29 (PA8)
- net Misc GPIO 1: now also J4.1 (Pin_1)
- net Button 4: now reaches U2.30 (PA9)
- net Button 4: now also J2.4 (Pin_4)
- net Button 2: now reaches U2.31 (PA10)
- net Button 2: now also J2.2 (Pin_2)
- net Button 1: now reaches U2.32 (PA11)
- net Button 1: now also J2.1 (Pin_1)
- net Button 3: now reaches U2.33 (PA12)
- net Button 3: now also J2.3 (Pin_3)
- no-connect marks 2 -> 11
Other:
- note removed: "0.3/0.45 mm vias for 4 layer board Default via size for two layer boards"
- note removed: "I2C pin configs: SDA: PF0, PA10, PA14, PB7, PB9 SCL: PF1, PA9, PA15, PB6, PB8"
- note removed: "Look at button schematic for Nucleo board"
- note removed: "VBAT supplies power to the real time clock when nothing is being supplied to VDD"
- moved on the sheet: D1, D2, D3, J1, R1, R12, R13, R2, R3

Commit message: finalized boards and cad files
Parts:
- added J13: Mux conn, symbol Connector:Conn_01x04_Socket
- C1, C4, C9: LCSC (none) -> C431646
- C5: footprint Capacitor_SMD:C_0805_2012Metric_Pad1.18x1.45mm_HandSolder -> Capacitor_SMD:C_0402_1005Metric_Pad0.74x0.62mm_HandSolder; LCSC (none) -> C431646
- H1, H2: value MountingHole -> MountingHole M3
- Q1, Q2, Q3, Q4, Q5: LCSC (none) -> C380910
- R1, R2, R3: value TBD -> 330R
- R10, R11, R7, R8, R9: LCSC (none) -> C2763787
- R12, R13: value TBD -> 10k
- R4: LCSC (none) -> C849802
- R6: LCSC (none) -> C311897
- U2: LCSC (none) -> C108516
Connections:
- net MUX1: now also J13.1 (Pin_1)
- net MUX2: now also J13.2 (Pin_2)
- net MUX3: now also J13.3 (Pin_3)
- net MUX4: now also J13.4 (Pin_4)
Other:
- moved on the sheet: H1, H2, J12, J2, J3, J4, J5

Commit message: added solderbridge for bootloader
Parts:
- added JP2: Solder Bridge, Jumper:SolderJumper-3_P1.3mm_Open_Pad1.0x1.5mm_NumberLabels, symbol Jumper:SolderJumper_3_Open
Connections:
- net GND: now also JP2.3 (B); no longer U2.44 (BOOT0)
- net VDD: now also JP2.1 (A)
- new net ~{BOOT}: JP2.2 (C), U2.44 (BOOT0)
Other:
- note added: "The BOOT0 pin should be shorted to ground under normal circumstances."
Changed lines of the file:
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@@
 	(wire
 		(pts
-			(xy 59.69 113.03) (xy 52.07 113.03)
+			(xy 25.4 93.98) (xy 25.4 97.79)
 		)
 		(stroke
@@
 	(wire
 		(pts
-			(xy 25.4 93.98) (xy 25.4 97.79)
+			(xy 36.83 167.64) (xy 36.83 172.72)
 		)
 		(stroke
@@
 	(wire
 		(pts
+			(xy 17.78 172.72) (xy 17.78 180.34)
+		)
+		(stroke
+			(width 0)
+			(type default)
+		)
+	)
+	(wire
+		(pts
 			(xy 38.1 120.65) (xy 38.1 121.92)
 		)
@@
 	(wire
 		(pts
-			(xy 52.07 113.03) (xy 52.07 114.3)
-		)
-		(stroke
-			(width 0)
-			(type default)
-		)
-	)
-	(wire
-		(pts
 			(xy 243.84 48.26) (xy 234.95 48.26)
 		)
@@
 	(wire
 		(pts
+			(xy 22.86 172.72) (xy 17.78 172.72)
+		)
+		(stroke
+			(width 0)
+			(type default)
+		)
+	)
+	(wire
+		(pts
 			(xy 226.06 48.26) (xy 234.95 48.26)
 		)
@@
 	(wire
 		(pts
+			(xy 54.61 113.03) (xy 59.69 113.03)
+		)
+		(stroke
+			(width 0)
+			(type default)
+		)
+	)
+	(wire
+		(pts
 			(xy 50.8 93.98) (xy 63.5 93.98)
 		)
@@
 	(wire
 		(pts
+			(xy 27.94 165.1) (xy 27.94 168.91)
+		)
+		(stroke
+			(width 0)
+			(type default)
+		)
+	)
+	(wire
+		(pts
 			(xy 92.71 133.35) (xy 97.79 133.35)
 		)
@@
 	(wire
 		(pts
+			(xy 36.83 172.72) (xy 33.02 172.72)
+		)
+		(stroke
+			(width 0)
+			(type default)
+		)
+	)
+	(wire
+		(pts
 			(xy 254 149.86) (xy 254 157.48)
 		)
@@
 		)
 	)
+	(text "The BOOT0 pin should be shorted to\nground under normal circumstances."
+		(exclude_from_sim no)
+		(at 33.528 189.738 0)
+		(effects
+			(font
+				(size 1.27 1.27)
+			)
+		)
+	)
 	(label "SDA"
 		(at 130.81 182.88 180)
@@
 		)
 	)
+	(label "~{BOOT}"
+		(at 54.61 113.03 180)
+		(fields_autoplaced yes)
+		(effects
+			(font
+				(size 1.27 1.27)
+			)
+			(justify right bottom)
+		)
+	)
 	(label "Button 5"
 		(at 97.79 107.95 0)
@@
 		)
 	)
+	(label "~{BOOT}"
+		(at 27.94 165.1 180)
+		(fields_autoplaced yes)
+		(effects
+			(font
+				(size 1.27 1.27)
+			)
+			(justify right bottom)
+		)
+	)
 	(label "SDA"
 		(at 54.61 158.75 180)
@@
 	(symbol
 		(lib_id "power:GND")
-		(at 52.07 114.3 0)
+		(at 17.78 180.34 0)
 		(unit 1)
 		(exclude_from_sim no)
@@
 		(dnp no)
 		(fields_autoplaced yes)
-		(property "Reference" "#PWR019"
-			(at 52.07 120.65 0)
+		(property "Reference" "#PWR061"
+			(at 17.78 186.69 0)
 			(effects
 				(font
@@
 		)
 		(property "Value" "GND"
-			(at 52.07 119.38 0)
+			(at 17.78 185.42 0)
 			(effects
 				(font
@@
 		)
 		(property "Footprint" ""
-			(at 52.07 114.3 0)
+			(at 17.78 180.34 0)
 			(effects
 				(font
@@
 		)
 		(property "Datasheet" ""
-			(at 52.07 114.3 0)
+			(at 17.78 180.34 0)
 			(effects
 				(font
@@
 		)
 		(property "Description" "Power symbol creates a global label with name \"GND\" , ground"
-			(at 52.07 114.3 0)
+			(at 17.78 180.34 0)
 			(effects
 				(font
@@
 			(project "led_2048"
 				(path "/c576df4b-92c0-44b0-b003-b697a5a04765/fbb28dfe-f4d8-4e18-86e7-4227759d21b0"
-					(reference "#PWR019")
+					(reference "#PWR061")
 					(unit 1)
 				)
@@
 	)
 	(symbol
+		(lib_id "power:VDD")
+		(at 36.83 167.64 0)
+		(unit 1)
+		(exclude_from_sim no)
+		(in_bom yes)
+		(on_board yes)
+		(dnp no)
+		(fields_autoplaced yes)
+		(property "Reference" "#PWR019"
+			(at 36.83 171.45 0)
+			(effects
+				(font
+					(size 1.27 1.27)
+				)
+				(hide yes)
+			)
+		)
+		(property "Value" "VDD"
+			(at 36.83 162.56 0)
+			(effects
+				(font
+					(size 1.27 1.27)
+				)
+			)
+		)
+		(property "Footprint" ""
+			(at 36.83 167.64 0)
+			(effects
+				(font
+					(size 1.27 1.27)
+				)
+				(hide yes)
+			)
+		)
+		(property "Datasheet" ""
+			(at 36.83 167.64 0)
+			(effects
+				(font
+					(size 1.27 1.27)
+				)
+				(hide yes)
+			)
+		)
+		(property "Description" "Power symbol creates a global label with name \"VDD\""
+			(at 36.83 167.64 0)
+			(effects
+				(font
+					(size 1.27 1.27)
+				)
+				(hide yes)
+			)
+		)
+		(pin "1"
+		)
+		(instances
+			(project "led_2048"
+				(path "/c576df4b-92c0-44b0-b003-b697a5a04765/fbb28dfe-f4d8-4e18-86e7-4227759d21b0"
+					(reference "#PWR019")
+					(unit 1)
+				)
+			)
+		)
+	)
+	(symbol
 		(lib_id "Connector:Conn_01x04_Socket")
 		(at 45.72 60.96 0)
@@
 					(unit 1)
 				)
+			)
+		)
+	)
+	(symbol
+		(lib_id "Jumper:SolderJumper_3_Open")
+		(at 27.94 172.72 180)
+		(unit 1)
+		(exclude_from_sim yes)
+		(in_bom no)
+		(on_board yes)
+		(dnp no)
+		(property "Reference" "JP2"
+			(at 27.94 179.07 0)
+			(effects
+				(font
+					(size 1.27 1.27)
+				)
+			)
+		)
+		(property "Value" "Solder Bridge"
+			(at 27.94 176.53 0)
+			(effects
+				(font
+					(size 1.27 1.27)
+				)
+			)
+		)
+		(property "Footprint" "Jumper:SolderJumper-3_P1.3mm_Open_Pad1.0x1.5mm_NumberLabels"
+			(at 27.94 172.72 0)
+			(effects
+				(font
+					(size 1.27 1.27)
+				)
+				(hide yes)
+			)
+		)
+		(property "Datasheet" "~"
+			(at 27.94 172.72 0)
+			(effects
+				(font
+					(size 1.27 1.27)
+				)
+				(hide yes)
+			)
+		)
+		(property "Description" "Solder Jumper, 3-pole, open"
+			(at 27.94 172.72 0)
+			(effects
+				(font
+					(size 1.27 1.27)
+				)
+				(hide yes)
+			)
+		)
+		(pin "3"
+		)
+		(pin "2"
+		)
+		(pin "1"
+		)
+		(instances
+			(project ""
+				(path "/c576df4b-92c0-44b0-b003-b697a5a04765/fbb28dfe-f4d8-4e18-86e7-4227759d21b0"
+					(reference "JP2")
+					(unit 1)
+				)

Commit message: minor schematic revisions
Parts:
- removed JP2: Solder Bridge, Jumper:SolderJumper-3_P1.3mm_Open_Pad1.0x1.5mm_NumberLabels, symbol Jumper:SolderJumper_3_Open
- added R12: 0R (DNP), Resistor_SMD:R_0805_2012Metric_Pad1.20x1.40mm_HandSolder, symbol Device:R_US
- added R13: 10k, Resistor_SMD:R_0805_2012Metric_Pad1.20x1.40mm_HandSolder, symbol Device:R_US
- renumbered J4 to J1, J1 to J2, J5 to J3, J12 to J4, J2 to J5, J3 to J6, J13 to J7, R12 to R14, R13 to R15
Connections:
- net GND: now also R13.2
- net VDD: now also R12.1
- net ~{BOOT}: now also R12.2, R13.1
