File: kicad/led_2048/seven_seg_display.kicad_sch (KiCad schematic)
At the start: 9 parts, among them U1 CL3641BH, U2 74HC595

Commit message: finished layout
Parts:
- added C11, C12: 0.1uF (DNP), Capacitor_SMD:C_0805_2012Metric_Pad1.18x1.45mm_HandSolder, symbol Device:C
- added J6: Power conn, Connector_PinSocket_2.00mm:PinSocket_1x02_P2.00mm_Vertical, symbol Connector:Conn_01x02_Socket
- added J7: Mux Conn, Connector_PinSocket_2.00mm:PinSocket_1x04_P2.00mm_Vertical, symbol Connector:Conn_01x04_Socket
- added J8: Shift Reg Conn, Connector_PinSocket_2.00mm:PinSocket_1x03_P2.00mm_Vertical, symbol Connector:Conn_01x03_Socket
- added J9: Misc conn 1, Connector_PinSocket_2.00mm:PinSocket_1x02_P2.00mm_Vertical, symbol Connector:Conn_01x02_Socket
- added R22, R23: 4.7k, Resistor_SMD:R_0805_2012Metric_Pad1.20x1.40mm_HandSolder, symbol Device:R_US
- added R24, R25: 100R (DNP), Resistor_SMD:R_0805_2012Metric_Pad1.20x1.40mm_HandSolder, symbol Device:R_US
- added SW3, SW4: Button, 2048_footprints:SW_TL1105SPF160Q, symbol Switch:SW_MEC_5E
Connections:
- net GND: now also J6.2 (Pin_2), R24.2, R25.2, SW3.1, SW3.2, SW4.1, SW4.2
- net Multiplex 1: now also J7.1 (Pin_1)
- net Multiplex 2: now also J7.2 (Pin_2)
- net Multiplex 3: now also J7.3 (Pin_3)
- net Multiplex 4: now also J7.4 (Pin_4)
- net Score clk: now also J8.1 (Pin_1)
- net Score data: now also J8.3 (Pin_3)
- net Score latch: now also J8.2 (Pin_2)
- net VDD: now also J6.1 (Pin_1), R22.2, R23.2
- new net: C11.2, R24.1
- new net: C12.2, R25.1
- new net Button 10: C12.1, J9.2 (Pin_2), R23.1, SW4.3 (K), SW4.4 (A)
- new net Button 9: C11.1, J9.1 (Pin_1), R22.1, SW3.3 (K), SW3.4 (A)

Commit message: finalized boards and cad files
Parts:
- R1, R2, R3, R4, R5, R6, R7: LCSC (none) -> C17557
- U2: LCSC (none) -> C18164493
Changed lines of the file:
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@@
+			)
+		)
+		(property "LCSC" "C17557"
+			(at 237.49 66.04 0)
+			(effects
+				(font
+					(size 1.27 1.27)
+				)
+				(hide yes)
 			)
 		)
@@
 			)
 		)
+		(property "LCSC" "C17557"
+			(at 217.17 66.04 0)
+			(effects
+				(font
+					(size 1.27 1.27)
+				)
+				(hide yes)
+			)
+		)
 		(pin "2"
 		)
@@
 			)
 		)
+		(property "LCSC" "C17557"
+			(at 237.49 93.98 0)
+			(effects
+				(font
+					(size 1.27 1.27)
+				)
+				(hide yes)
+			)
+		)
 		(pin "2"
 		)
@@
 			)
 		)
+		(property "LCSC" "C17557"
+			(at 217.17 93.98 0)
+			(effects
+				(font
+					(size 1.27 1.27)
+				)
+				(hide yes)
+			)
+		)
 		(pin "2"
 		)
@@
 			)
 		)
+		(property "LCSC" "C17557"
+			(at 207.01 93.98 0)
+			(effects
+				(font
+					(size 1.27 1.27)
+				)
+				(hide yes)
+			)
+		)
 		(pin "2"
 		)
@@
 			)
 		)
+		(property "LCSC" "C18164493"
+			(at 191.77 82.55 0)
+			(effects
+				(font
+					(size 1.27 1.27)
+				)
+				(hide yes)
+			)
+		)
 		(pin "6"
 		)
@@
 			)
 		)
+		(property "LCSC" "C17557"
+			(at 227.33 66.04 0)
+			(effects
+				(font
+					(size 1.27 1.27)
+				)
+				(hide yes)
+			)
+		)
 		(pin "2"
 		)
@@
 			(at 227.33 93.98 0)
 			(effects
+				(font
+					(size 1.27 1.27)
+				)
+				(hide yes)
+			)
+		)
+		(property "LCSC" "C17557"
+			(at 227.33 93.98 0)
+			(effects

Commit message: minor schematic revisions
Parts:
- renumbered J8 to J10, J9 to J11, J6 to J8, J7 to J9, R22 to R24, R23 to R25, R24 to R26, R25 to R27
Changed lines of the file:
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@@
 			(project "seven_seg_display"
 				(path "/c576df4b-92c0-44b0-b003-b697a5a04765/b7eda4aa-318d-4020-9d5c-8e21103c3223"
-					(reference "R17")
+					(reference "R19")
 					(unit 1)
 				)
@@
 			(project "seven_seg_display"
 				(path "/c576df4b-92c0-44b0-b003-b697a5a04765/b7eda4aa-318d-4020-9d5c-8e21103c3223"
-					(reference "R15")
+					(reference "R17")
 					(unit 1)
 				)
@@
 		(on_board yes)
 		(dnp no)
-		(property "Reference" "J9"
+		(property "Reference" "J11"
 			(at 93.98 63.5 0)
 			(effects
@@
 			(project "led_2048"
 				(path "/c576df4b-92c0-44b0-b003-b697a5a04765/b7eda4aa-318d-4020-9d5c-8e21103c3223"
-					(reference "J9")
+					(reference "J11")
 					(unit 1)
 				)
@@
 		(dnp no)
 		(fields_autoplaced yes)
-		(property "Reference" "#PWR039"
+		(property "Reference" "#PWR040"
 			(at 62.23 143.51 0)
 			(effects
@@
 			(project "led_2048"
 				(path "/c576df4b-92c0-44b0-b003-b697a5a04765/b7eda4aa-318d-4020-9d5c-8e21103c3223"
-					(reference "#PWR039")
+					(reference "#PWR040")
 					(unit 1)
 				)
@@
 		(dnp no)
 		(fields_autoplaced yes)
-		(property "Reference" "#PWR036"
+		(property "Reference" "#PWR037"
 			(at 177.8 71.12 0)
 			(effects
@@
 			(project ""
 				(path "/c576df4b-92c0-44b0-b003-b697a5a04765/b7eda4aa-318d-4020-9d5c-8e21103c3223"
-					(reference "#PWR036")
+					(reference "#PWR037")
 					(unit 1)
 				)
@@
 		(on_board yes)
 		(dnp no)
-		(property "Reference" "R24"
+		(property "Reference" "R26"
 			(at 52.07 158.75 90)
 			(effects
@@
 			(project "led_2048"
 				(path "/c576df4b-92c0-44b0-b003-b697a5a04765/b7eda4aa-318d-4020-9d5c-8e21103c3223"
-					(reference "R24")
+					(reference "R26")
 					(unit 1)
 				)
@@
 			(project "seven_seg_display"
 				(path "/c576df4b-92c0-44b0-b003-b697a5a04765/b7eda4aa-318d-4020-9d5c-8e21103c3223"
-					(reference "R21")
+					(reference "R23")
 					(unit 1)
 				)
@@
 			(project "seven_seg_display"
 				(path "/c576df4b-92c0-44b0-b003-b697a5a04765/b7eda4aa-318d-4020-9d5c-8e21103c3223"
-					(reference "#PWR037")
+					(reference "#PWR038")
 					(unit 1)
 				)
@@
 			(project "seven_seg_display"
 				(path "/c576df4b-92c0-44b0-b003-b697a5a04765/b7eda4aa-318d-4020-9d5c-8e21103c3223"
-					(reference "R19")
+					(reference "R21")
 					(unit 1)
 				)
@@
 			(project "seven_seg_display"
 				(path "/c576df4b-92c0-44b0-b003-b697a5a04765/b7eda4aa-318d-4020-9d5c-8e21103c3223"
-					(reference "R18")
+					(reference "R20")
 					(unit 1)
 				)
@@
 		(dnp no)
 		(fields_autoplaced yes)
-		(property "Reference" "#PWR042"
+		(property "Reference" "#PWR043"
 			(at 92.71 175.26 0)
 			(effects
@@
 			(project "led_2048"
 				(path "/c576df4b-92c0-44b0-b003-b697a5a04765/b7eda4aa-318d-4020-9d5c-8e21103c3223"
-					(reference "#PWR042")
+					(reference "#PWR043")
 					(unit 1)
 				)
@@
 		(dnp no)
 		(fields_autoplaced yes)
-		(property "Reference" "#PWR040"
+		(property "Reference" "#PWR041"
 			(at 111.76 143.51 0)
 			(effects
@@
 			(project "led_2048"
 				(path "/c576df4b-92c0-44b0-b003-b697a5a04765/b7eda4aa-318d-4020-9d5c-8e21103c3223"
-					(reference "#PWR040")
+					(reference "#PWR041")
 					(unit 1)
 				)
@@
 		(on_board yes)
 		(dnp no)
-		(property "Reference" "R23"
+		(property "Reference" "R25"
 			(at 116.84 144.78 0)
 			(effects
@@
 			(project "led_2048"
 				(path "/c576df4b-92c0-44b0-b003-b697a5a04765/b7eda4aa-318d-4020-9d5c-8e21103c3223"
-					(reference "R23")
+					(reference "R25")
 					(unit 1)
 				)
@@
 			(project ""
 				(path "/c576df4b-92c0-44b0-b003-b697a5a04765/b7eda4aa-318d-4020-9d5c-8e21103c3223"
-					(reference "#PWR038")
+					(reference "#PWR039")
 					(unit 1)
 				)
@@
 		(dnp no)
 		(fields_autoplaced yes)
-		(property "Reference" "J8"
+		(property "Reference" "J10"
 			(at 92.71 52.0699 0)
 			(effects
@@
 			(project ""
 				(path "/c576df4b-92c0-44b0-b003-b697a5a04765/b7eda4aa-318d-4020-9d5c-8e21103c3223"
-					(reference "J8")
+					(reference "J10")
 					(unit 1)
 				)
@@
 		(dnp no)
 		(fields_autoplaced yes)
-		(property "Reference" "#PWR041"
+		(property "Reference" "#PWR042"
 			(at 43.18 175.26 0)
 			(effects
@@
 			(project "led_2048"
 				(path "/c576df4b-92c0-44b0-b003-b697a5a04765/b7eda4aa-318d-4020-9d5c-8e21103c3223"
-					(reference "#PWR041")
+					(reference "#PWR042")
 					(unit 1)
 				)
@@
 		(dnp no)
 		(fields_autoplaced yes)
-		(property "Reference" "#PWR034"
+		(property "Reference" "#PWR035"
 			(at 35.56 53.34 0)
 			(effects
@@
 			(project "led_2048"
 				(path "/c576df4b-92c0-44b0-b003-b697a5a04765/b7eda4aa-318d-4020-9d5c-8e21103c3223"
-					(reference "#PWR034")
+					(reference "#PWR035")
 					(unit 1)
 				)
@@
 		(dnp no)
 		(fields_autoplaced yes)
-		(property "Reference" "#PWR035"
+		(property "Reference" "#PWR036"
 			(at 191.77 66.04 0)
 			(effects
@@
 			(project "led_2048"
 				(path "/c576df4b-92c0-44b0-b003-b697a5a04765/b7eda4aa-318d-4020-9d5c-8e21103c3223"
-					(reference "#PWR035")
+					(reference "#PWR036")
 					(unit 1)
 				)
@@
 		(on_board yes)
 		(dnp no)
-		(property "Reference" "J6"
+		(property "Reference" "J8"
 			(at 46.99 39.37 0)
 			(effects
@@
 			(project "led_2048"
 				(path "/c576df4b-92c0-44b0-b003-b697a5a04765/b7eda4aa-318d-4020-9d5c-8e21103c3223"
-					(reference "J6")
+					(reference "J8")
 					(unit 1)
 				)
@@
 		(dnp no)
 		(fields_autoplaced yes)
-		(property "Reference" "#PWR033"
+		(property "Reference" "#PWR034"
 			(at 35.56 38.1 0)
 			(effects
@@
 			(project "led_2048"
 				(path "/c576df4b-92c0-44b0-b003-b697a5a04765/b7eda4aa-318d-4020-9d5c-8e21103c3223"
-					(reference "#PWR033")
+					(reference "#PWR034")
 					(unit 1)
 				)
@@
 		(on_board yes)
 		(dnp no)
-		(property "Reference" "R25"
+		(property "Reference" "R27"
 			(at 101.6 158.75 90)
 			(effects
@@
 			(project "led_2048"
 				(path "/c576df4b-92c0-44b0-b003-b697a5a04765/b7eda4aa-318d-4020-9d5c-8e21103c3223"
-					(reference "R25")
+					(reference "R27")
 					(unit 1)
 				)
@@
 		(on_board yes)
 		(dnp no)
-		(property "Reference" "R22"
+		(property "Reference" "R24"
 			(at 67.31 144.78 0)
 			(effects
@@
 			(project "led_2048"
 				(path "/c576df4b-92c0-44b0-b003-b697a5a04765/b7eda4aa-318d-4020-9d5c-8e21103c3223"
-					(reference "R22")
+					(reference "R24")
 					(unit 1)
 				)
@@
 			(project "seven_seg_display"
 				(path "/c576df4b-92c0-44b0-b003-b697a5a04765/b7eda4aa-318d-4020-9d5c-8e21103c3223"
-					(reference "R16")
+					(reference "R18")
 					(unit 1)
 				)
@@
 			(project "seven_seg_display"
 				(path "/c576df4b-92c0-44b0-b003-b697a5a04765/b7eda4aa-318d-4020-9d5c-8e21103c3223"
-					(reference "R20")
+					(reference "R22")
 					(unit 1)
 				)
@@
 		(dnp no)
 		(fields_autoplaced yes)
-		(property "Reference" "J7"
+		(property "Reference" "J9"
 			(at 92.71 39.3699 0)
 			(effects
@@
 			(project ""
 				(path "/c576df4b-92c0-44b0-b003-b697a5a04765/b7eda4aa-318d-4020-9d5c-8e21103c3223"
-					(reference "J7")
-					(unit 1)
-				)
+					(reference "J9")
+					(unit 1)
+				)
